File: zulu-ctrl-board-v1.0-kicad/ctrl_board.kicad_sch (KiCad schematic)
At the start: 36 parts, among them J1 Zulu I2C w/ interrupt Connect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, J2 OLED Connector, J3 Conn_01x06_Odd_Even, J305 I2C Qwiic, J4 Aux GPIO Connector, J5 CENTER_INT, J8 Zulu I2C w/ interrupt Connect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, SW1 SW_SPST, SW2 SW_SPST, SW4 Rotary_Encoder_Switch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

Commit message: Layout done for the Zulu Control Board v1.0
Layout done for revision 2023a.
Parts:
- removed G1, G2: Pi Logo, mousebites:pi_logo, symbol graphics:Generic_Graphic
- removed G3: KiCad Logo, Symbol:KiCad-Logo2_5mm_SilkScreen, symbol graphics:Generic_Graphic
- removed G4: DogCow, mousebites:dogcow, symbol graphics:Generic_Graphic
- removed J3: Conn_01x06_Odd_Even, Connector_PinHeader_2.54mm:PinHeader_1x06_P2.54mm_Vertical, symbol Connector_Generic:Conn_01x06
- removed J4: Aux GPIO Connector, Connector_PinHeader_2.54mm:PinHeader_1x02_P2.54mm_Vertical, symbol Connector_Generic:Conn_01x02
- added D1, D2, D3: LED, LED_THT:LED_D5.0mm, symbol Device:LED
- added R14: 10k, Resistor_SMD:R_0805_2012Metric, symbol Device:R_Small
- J305: footprint Connector_JST:JST_SH_SM04B-SRSS-TB_1x04-1MP_P1.00mm_Horizontal -> mousebites:JST_SH_SM04B-SRSS-TB_1x04-1MP_P1.00mm_Horizontal
Connections:
- net +3V3: now also R13.2, R14.2; no longer R13.1
- net LED_1: now also D1.1 (K)
- net LED_2: now also D2.1 (K)
- net at R12.2: now also D1.2 (A)
- net BUTTON_3 renamed LED_3
- net LED_3: now also D3.1 (K)
- new net: D2.2 (A), R13.1
- new net: D3.2 (A), R14.1
- no-connect marks 3 -> 2
Other:
- note added: "OLED Display"
- moved on the sheet: J2, R12, R13

Commit message: JLCPCB fixes
Fixed rotation of GPIO expansion IC.
Modified GitHub workflow
Parts:
- U1: JLCPCBCORRECT (none) -> 0;0;-90
Changed lines of the file:
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@@
+      (effects (font (size 1.27 1.27)) hide)
+    )
+    (property "JLCPCBCORRECT" "" (at 52.07 114.3 0)
       (effects (font (size 1.27 1.27)) hide)
     )
@@
       (effects (font (size 1.27 1.27)) hide)
     )
+    (property "JLCPCBCORRECT" "" (at 91.44 96.52 0)
+      (effects (font (size 1.27 1.27)) hide)
+    )
     (pin "1")
     (pin "2")
@@
       (effects (font (size 1.27 1.27)) hide)
     )
+    (property "JLCPCBCORRECT" "" (at 91.44 106.68 0)
+      (effects (font (size 1.27 1.27)) hide)
+    )
     (pin "1")
     (pin "2")
@@
       (effects (font (size 1.27 1.27)) hide)
     )
+    (property "JLCPCBCORRECT" "" (at 106.68 93.98 0)
+      (effects (font (size 1.27 1.27)) hide)
+    )
     (pin "1")
     (pin "2")
@@
       (effects (font (size 1.27 1.27)) hide)
     )
+    (property "JLCPCBCORRECT" "" (at 106.68 104.14 0)
+      (effects (font (size 1.27 1.27)) hide)
+    )
     (pin "1")
     (pin "2")
@@
       (effects (font (size 1.27 1.27)) hide)
     )
+    (property "JLCPCBCORRECT" "" (at 39.37 134.62 0)
+      (effects (font (size 1.27 1.27)) hide)
+    )
     (pin "1")
     (pin "2")
@@
       (effects (font (size 1.27 1.27)) hide)
     )
+    (property "JLCPCBCORRECT" "" (at 39.37 137.16 0)
+      (effects (font (size 1.27 1.27)) hide)
+    )
     (pin "1")
     (pin "2")
@@
     )
     (property "Datasheet" "~" (at 92.71 135.636 0)
+      (effects (font (size 1.27 1.27)) hide)
+    )
+    (property "JLCPCBCORRECT" "" (at 92.71 142.24 0)
       (effects (font (size 1.27 1.27)) hide)
     )
@@
       (effects (font (size 1.27 1.27)) hide)
     )
+    (property "JLCPCBCORRECT" "" (at 172.72 22.86 0)
+      (effects (font (size 1.27 1.27)) hide)
+    )
     (pin "1")
     (pin "2")
@@
       (effects (font (size 1.27 1.27)) hide)
     )
+    (property "JLCPCBCORRECT" "" (at 106.68 135.89 0)
+      (effects (font (size 1.27 1.27)) hide)
+    )
     (pin "1")
     (pin "2")
@@
       (effects (font (size 1.27 1.27)) hide)
     )
+    (property "JLCPCBCORRECT" "" (at 240.665 75.565 0)
+      (effects (font (size 1.27 1.27)) hide)
+    )
     (pin "1")
     (pin "2")
@@
       (effects (font (size 1.27 1.27)) hide)
     )
+    (property "JLCPCBCORRECT" "" (at 235.585 75.565 0)
+      (effects (font (size 1.27 1.27)) hide)
+    )
     (pin "1")
     (pin "2")
@@
       (effects (font (size 1.27 1.27)) hide)
     )
+    (property "JLCPCBCORRECT" "" (at 55.88 135.89 0)
+      (effects (font (size 1.27 1.27)) hide)
+    )
     (pin "1")
     (pin "2")
@@
       (effects (font (size 1.27 1.27)) hide)
     )
+    (property "JLCPCBCORRECT" "" (at 62.23 135.89 0)
+      (effects (font (size 1.27 1.27)) hide)
+    )
     (pin "1")
     (pin "2")
@@
     )
     (property "Datasheet" "~" (at 57.785 169.545 0)
+      (effects (font (size 1.27 1.27)) hide)
+    )
+    (property "JLCPCBCORRECT" "" (at 57.785 169.545 0)
       (effects (font (size 1.27 1.27)) hide)
     )
@@
     (property "SUPPLIER" "NXP" (at 203.2 34.29 0)
       (effects (font (size 1.27 1.27)) (justify left bottom) hide)
+    )
+    (property "JLCPCBCORRECT" "0;0;-90" (at 203.2 34.29 0)
+      (effects (font (size 1.27 1.27)) hide)
     )
     (pin "1")
@@
       (effects (font (size 1.27 1.27)) hide)
     )
+    (property "JLCPCBCORRECT" "" (at 232.41 26.67 0)
+      (effects (font (size 1.27 1.27)) hide)
+    )
     (pin "1")
     (pin "2")
@@
       (effects (font (size 1.27 1.27)) hide)
     )
+    (property "JLCPCBCORRECT" "" (at 147.32 55.88 0)
+      (effects (font (size 1.27 1.27)) hide)
+    )
     (pin "1")
     (pin "2")
@@
       (effects (font (size 1.27 1.27)) hide)
     )
+    (property "JLCPCBCORRECT" "" (at 160.02 55.88 0)
+      (effects (font (size 1.27 1.27)) hide)
+    )
     (pin "1")
     (pin "2")
@@
       (effects (font (size 1.27 1.27)) hide)
     )
+    (property "JLCPCBCORRECT" "" (at 171.45 55.88 0)
+      (effects (font (size 1.27 1.27)) hide)
+    )
     (pin "1")
     (pin "2")
@@
       (effects (font (size 1.27 1.27)) hide)
     )
+    (property "JLCPCBCORRECT" "" (at 166.37 41.91 0)
+      (effects (font (size 1.27 1.27)) hide)
+    )
     (pin "1")
     (pin "2")
@@
       (effects (font (size 1.27 1.27)) hide)
     )
+    (property "JLCPCBCORRECT" "" (at 177.8 44.45 0)
+      (effects (font (size 1.27 1.27)) hide)
+    )
     (pin "1")
     (pin "2")
@@
       (effects (font (size 1.27 1.27)) hide)
     )
+    (property "JLCPCBCORRECT" "" (at 152.4 39.37 0)
+      (effects (font (size 1.27 1.27)) hide)
+    )
     (pin "1")
     (pin "2")
@@
     )
     (property "Datasheet" "~" (at 236.855 90.17 0)
+      (effects (font (size 1.27 1.27)) hide)
+    )
+    (property "JLCPCBCORRECT" "" (at 236.855 90.17 0)
       (effects (font (size 1.27 1.27)) hide)
     )
@@
     )
     (property "LCSC" "N/A" (at 252.73 111.125 0)
+      (effects (font (size 1.27 1.27)) hide)
+    )
+    (property "JLCPCBCORRECT" "" (at 252.73 111.125 0)
       (effects (font (size 1.27 1.27)) hide)
     )
@@
       (effects (font (size 1.27 1.27)) hide)
     )
+    (property "JLCPCBCORRECT" "" (at 173.99 151.765 0)
+      (effects (font (size 1.27 1.27)) hide)
+    )
     (pin "1")
     (pin "2")
@@
       (effects (font (size 1.27 1.27)) hide)
     )
+    (property "JLCPCBCORRECT" "" (at 248.92 76.2 0)
+      (effects (font (size 1.27 1.27)) hide)
+    )
     (pin "1")
     (pin "2")
@@
     )
     (property "Datasheet" "~" (at 227.33 80.645 0)
+      (effects (font (size 1.27 1.27)) hide)
+    )
+    (property "JLCPCBCORRECT" "" (at 227.33 80.645 0)
       (effects (font (size 1.27 1.27)) hide)
     )
@@
       (effects (font (size 1.27 1.27)) hide)
     )
+    (property "JLCPCBCORRECT" "" (at 74.93 182.88 0)
+      (effects (font (size 1.27 1.27)) hide)
+    )
     (pin "1")
     (instances
@@
     )
     (property "Datasheet" "~" (at 231.775 85.09 0)
+      (effects (font (size 1.27 1.27)) hide)
+    )
+    (property "JLCPCBCORRECT" "" (at 231.775 85.09 0)
       (effects (font (size 1.27 1.27)) hide)
     )
@@
       (effects (font (size 1.27 1.27)) hide)
     )
+    (property "JLCPCBCORRECT" "" (at 51.435 83.82 0)
+      (effects (font (size 1.27 1.27)) hide)
+    )
     (pin "1")
     (instances
@@
     )
     (property "LCSC" "C17414" (at 226.06 22.86 0)
+      (effects (font (size 1.27 1.27)) hide)
+    )
+    (property "JLCPCBCORRECT" "" (at 226.06 22.86 0)
       (effects (font (size 1.27 1.27)) hide)
     )
@@
       (effects (font (size 1.27 1.27)) hide)
     )
+    (property "JLCPCBCORRECT" "" (at 85.725 182.88 0)
+      (effects (font (size 1.27 1.27)) hide)
+    )
     (pin "1")
     (instances
@@
       (effects (font (size 1.27 1.27)) hide)
     )
+    (property "JLCPCBCORRECT" "" (at 252.73 142.875 0)
+      (effects (font (size 1.27 1.27)) hide)
+    )
